File: pcbschem/pcbschem/pcbschem.kicad_pcb (KiCad board)
At the start: 2 copper layers, 50.8 x 22.9 mm, 65 parts, among them IC1 RP2040_QFN56, Q3 DMG341, SW1 KMR2, SW2 KMR2, U1 2MB Flash, U1 MPU-9250, U2 AP2112-3.3, U3 MCP73831T-2ACI/OT, X1 JSTPH, X6 USB Type C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

Commit message: update stuff
Parts:
- removed JP1: , 1X16_ROUND
- removed JP3: , 1X12_ROUND
- removed U$28: , ADAFRUIT_3.5MM
Routing:
- net (no net): track 1294.4 -> 1025.5 mm, vias 92 -> 85
Other:
- board text removed: "A&G"
- board text removed: "AD0 SDO"
- board text removed: "AUXCL"
- board text removed: "AUXDA"
- board text removed: "FSYNC"
- board text removed: "VDD"
- board text removed: "VDDIO"
- board text removed: "X"
- board text removed: "Y"
- board text removed: "Z"

Commit message: e
Parts:
- removed SJ1: JUMPER-PAD-2-NC_BY_PASTEFULL-BOX-SILK, PAD-JUMPER-2-NC_BY_PASTE_YES_SILK_FULL_BOX
- removed SJ2: JUMPER_PAD-3-1&2_NC_BY_PASTE, PAD-HUMPER-3-1&2_NC_BY_PASTE_YES_SILK_FULL_BOX
- removed the SW2 at (145.8, 101.3)
- removed the SW2 at (145.7, 105.5)
- added SW3: KMR2, BTN_KMR2_4.6X2.8, F.Cu at (228.9, 123.6)
- added SW4: KMR2, BTN_KMR2_4.6X2.8, F.Cu at (228.9, 119.5)
- moved @HOLE0 85.1 mm to (254.5, 113.0)
- moved C1 85.1 mm to (220.2, 123.6)
- moved C13 85.1 mm to (238.7, 127.6)
- moved C14 85.1 mm to (240.2, 115.6)
- moved C2 85.1 mm to (234.5, 114.9)
- moved C6 85.1 mm to (255.2, 128.5)
- moved CHG 85.1 mm to (208.0, 127.9)
- moved D+1 85.1 mm to (207.7, 123.1)
- moved D-1 85.1 mm to (207.6, 120.5)
- moved D4 85.1 mm to (218.2, 121.1)
- moved R11 85.1 mm to (251.9, 115.1)
- moved R2 85.1 mm to (212.0, 128.8)
- moved R3 85.1 mm to (225.2, 121.9)
- moved R4 85.1 mm to (228.1, 114.9)
- moved R5 85.1 mm to (251.9, 118.1)
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- renumbered C1 to C18, C2 to C6, R1 to R14, R2 to R15, R3 to R16, U1 to U4
Routing:
- net (no net): track 1025.5 -> 1065.9 mm, vias 85 -> 84
Other:
- rule via_min_size: 0.4 -> 0.1524
